Commit message: first demo with franka robot on GPU with sapien

File: furniture_bench/assets_no_tags/furniture/urdf/lamp/lamp_base.urdf (robot description, URDF)
Before this commit: robot lamp_base, 1 links, 0 joints
Links:
- link lamp_base: geometry collision mesh filename=../../mesh/lamp/lamp_base.obj scale=1 1 1; visual mesh filename=../../mesh/lamp/lamp_base.obj scale=1 1 1

File: furniture_bench/assets_no_tags/furniture/urdf/lamp/lamp_bulb.urdf (robot description, URDF)
Before this commit: robot lamp_bulb, 1 links, 0 joints
Links:
- link lamp_bulb: geometry collision mesh filename=../../mesh/lamp/lamp_bulb.obj scale=1 1 1; visual mesh filename=../../mesh/lamp/lamp_bulb.obj scale=1 1 1

File: furniture_bench/assets_no_tags/furniture/urdf/lamp/lamp_hood.urdf (robot description, URDF)
Before this commit: robot lamp_hood, 1 links, 0 joints
Links:
- link lamp_hood: geometry collision mesh filename=../../mesh/lamp/lamp_hood.obj scale=1 1 1; visual mesh filename=../../mesh/lamp/lamp_hood.obj scale=1 1 1

Commit message: basic implementation of reset & Bugfix observation reading of position (considering scene offset)

File: furniture_bench/assets_no_tags/furniture/urdf/lamp/lamp_base.urdf (robot description, URDF)
Before this commit: robot lamp_base, 1 links, 0 joints
Links:
- link lamp_base: geometry collision mesh filename=../mesh/lamp/lamp_base.obj scale=1 1 1; visual mesh filename=../mesh/lamp/lamp_base.obj scale=1 1 1

File: furniture_bench/assets_no_tags/furniture/urdf/lamp/lamp_bulb.urdf (robot description, URDF)
Before this commit: robot lamp_bulb, 1 links, 0 joints
Links:
- link lamp_bulb: geometry collision mesh filename=../mesh/lamp/lamp_bulb.obj scale=1 1 1; visual mesh filename=../mesh/lamp/lamp_bulb.obj scale=1 1 1

File: furniture_bench/assets_no_tags/furniture/urdf/lamp/lamp_hood.urdf (robot description, URDF)
Before this commit: robot lamp_hood, 1 links, 0 joints
Links:
- link lamp_hood: geometry collision mesh filename=../mesh/lamp/lamp_hood.obj scale=1 1 1; visual mesh filename=../mesh/lamp/lamp_hood.obj scale=1 1 1

File: furniture_bench/assets_no_tags/furniture/urdf/square_table/square_table_leg1.urdf (robot description, URDF)
Before this commit: robot square_table_leg1, 1 links, 0 joints
Links:
- link square_table_leg1: geometry collision mesh filename=../../mesh/square_table/square_table_leg1.obj scale=1 1 1; visual mesh filename=../../mesh/square_table/square_table_leg1.obj scale=1 1 1

File: furniture_bench/assets_no_tags/furniture/urdf/square_table/square_table_leg2.urdf (robot description, URDF)
Before this commit: robot square_table_leg2, 1 links, 0 joints
Links:
- link square_table_leg2: geometry collision mesh filename=../../mesh/square_table/square_table_leg2.obj scale=1 1 1; visual mesh filename=../../mesh/square_table/square_table_leg2.obj scale=1 1 1

File: furniture_bench/assets_no_tags/furniture/urdf/square_table/square_table_leg3.urdf (robot description, URDF)
Before this commit: robot square_table_leg3, 1 links, 0 joints
Links:
- link square_table_leg3: geometry collision mesh filename=../../mesh/square_table/square_table_leg3.obj scale=1 1 1; visual mesh filename=../../mesh/square_table/square_table_leg3.obj scale=1 1 1

File: furniture_bench/assets_no_tags/furniture/urdf/square_table/square_table_leg4.urdf (robot description, URDF)
Before this commit: robot square_table_leg4, 1 links, 0 joints
Links:
- link square_table_leg4: geometry collision mesh filename=../../mesh/square_table/square_table_leg4.obj scale=1 1 1; visual mesh filename=../../mesh/square_table/square_table_leg4.obj scale=1 1 1

File: furniture_bench/assets_no_tags/furniture/urdf/square_table/square_table_top.urdf (robot description, URDF)
Before this commit: robot square_top, 1 links, 0 joints
Links:
- link square_top: geometry collision mesh filename=../../mesh/square_table/square_table_top.obj scale=1 1 1; visual mesh filename=../../mesh/square_table/square_table_top.obj scale=1 1 1
