Commit message: Bugfix for parallel rendering and simulation

File: furniture_bench/assets_no_tags/furniture/urdf/lamp/lamp_bulb.urdf (robot description, URDF)
Before this commit: robot lamp_bulb, 1 links, 0 joints
Links:
- link lamp_bulb: geometry collision mesh filename=../mesh/lamp/lamp_bulb.obj scale=1 1 1; visual mesh filename=../../mesh/lamp/lamp_bulb.obj scale=1 1 1
