Commit message: Test with teleop

File: furniture_bench/assets/furniture/urdf/round_table/round_table_base.urdf (robot description, URDF)
Before this commit: robot round_table_base, 1 links, 0 joints
Links:
- link round_table_base: geometry collision mesh filename=../../mesh/round_table/round_table_base.obj scale=1 1 1; visual mesh filename=../../mesh/round_table/round_table_base.obj scale=1 1 1

File: furniture_bench/assets/furniture/urdf/round_table/round_table_top.urdf (robot description, URDF)
Before this commit: robot round_table_top, 1 links, 0 joints
Links:
- link round_table_top: geometry collision mesh filename=../../mesh/round_table/round_table_top.obj scale=1 1 1; visual mesh filename=../../mesh/round_table/round_table_top.obj scale=1 1 1

File: furniture_bench/assets_no_tags/furniture/urdf/lamp/lamp_bulb.urdf (robot description, URDF)
Before this commit: robot lamp_bulb, 1 links, 0 joints
Links:
- link lamp_bulb: geometry collision mesh filename=../../mesh/lamp/lamp_bulb.obj scale=1 1 1; visual mesh filename=../../mesh/lamp/lamp_bulb.obj scale=1 1 1

File: furniture_bench/assets_no_tags/furniture/urdf/round_table/round_table_leg.urdf (robot description, URDF)
Before this commit: robot round_table_leg, 1 links, 0 joints
Links:
- link round_table_leg: geometry collision mesh filename=../../mesh/round_table/round_table_leg.obj scale=1 1 1; visual mesh filename=../../mesh/round_table/round_table_leg.obj scale=1 1 1

File: furniture_bench/assets_no_tags/furniture/urdf/stool/stool_leg2.urdf (robot description, URDF)
Before this commit: robot stool_leg2, 1 links, 0 joints
Links:
- link stool_leg2: geometry collision mesh filename=../../mesh/stool/stool_leg2.obj scale=1 1 1; visual mesh filename=../../mesh/stool/stool_leg2.obj scale=1 1 1

File: furniture_bench/assets_no_tags/furniture/urdf/stool/stool_leg3.urdf (robot description, URDF)
Before this commit: robot stool_leg3, 1 links, 0 joints
Links:
- link stool_leg3: geometry collision mesh filename=../../mesh/stool/stool_leg3.obj scale=1 1 1; visual mesh filename=../../mesh/stool/stool_leg3.obj scale=1 1 1

File: furniture_bench/assets_no_tags/furniture/urdf/stool/stool_seat.urdf (robot description, URDF)
Before this commit: robot stool_seat, 1 links, 0 joints
Links:
- link stool_seat: geometry collision mesh filename=../../mesh/stool/stool_seat.obj scale=1 1 1; visual mesh filename=../../mesh/stool/stool_seat.obj scale=1 1 1
