Commit message: fix(mug_rack)

File: furniture_bench/assets_no_tags/furniture/scans/urdf/mug_rack/mug.urdf (robot description, URDF)
Before this commit: robot mug, 1 links, 0 joints
Links:
- link mug: geometry collision mesh filename=../../mesh/mug_rack/muggood/muggood.obj scale=1 1 1; visual mesh filename=../../mesh/mug_rack/muggood/muggood.obj scale=1 1 1

File: furniture_bench/assets_no_tags/furniture/scans/urdf/mug_rack/rack.urdf (robot description, URDF)
Before this commit: robot rack, 1 links, 0 joints
Links:
- link rack: geometry collision mesh filename=../../mesh/mug_rack/mugrack2/mugrack2.obj scale=1 1 1; visual mesh filename=../../mesh/mug_rack/mugrack2/mugrack2.obj scale=1 1 1
